Commit message: Fixed cottage package name references

File: gazebo/src/cottage/urdf/cottage_blender_Cube.urdf.xacro (robot description, xacro)
@@ -9,5 +9,5 @@
       <origin xyz="0 0 0" rpy="0 0 0" />
       <geometry>
-        <mesh filename="package://cottage_gazebo/meshes/cottage_blender_Cube.dae" />
+        <mesh filename="package://cottage/meshes/cottage_blender_Cube.dae" />
       </geometry>
     </visual>
@@ -15,5 +15,5 @@
       <origin xyz="0 0 0" rpy="0 0 0" />
       <geometry>
-        <mesh filename="package://cottage_gazebo/meshes/cottage_blender_Cube.dae" />
+        <mesh filename="package://cottage/meshes/cottage_blender_Cube.dae" />
       </geometry>
     </collision>

File: gazebo/src/cottage/urdf/cottage_blender_ground.urdf.xacro (robot description, xacro)
@@ -9,5 +9,5 @@
       <origin xyz="0 0 0" rpy="0 0 0" />
       <geometry>
-        <mesh filename="package://cottage_gazebo/meshes/cottage_blender_ground.dae" />
+        <mesh filename="package://cottage/meshes/cottage_blender_ground.dae" />
       </geometry>
     </visual>
@@ -15,5 +15,5 @@
       <origin xyz="0 0 0" rpy="0 0 0" />
       <geometry>
-        <mesh filename="package://cottage_gazebo/meshes/cottage_blender_ground.dae" />
+        <mesh filename="package://cottage/meshes/cottage_blender_ground.dae" />
       </geometry>
     </collision>

File: gazebo/src/cottage/urdf/cottage_blender_light_1.urdf.xacro (robot description, xacro)
@@ -9,5 +9,5 @@
       <origin xyz="0 0 0" rpy="0 0 0" />
       <geometry>
-        <mesh filename="package://cottage_gazebo/meshes/cottage_blender_light_1.dae" />
+        <mesh filename="package://cottage/meshes/cottage_blender_light_1.dae" />
       </geometry>
     </visual>
@@ -15,5 +15,5 @@
       <origin xyz="0 0 0" rpy="0 0 0" />
       <geometry>
-        <mesh filename="package://cottage_gazebo/meshes/cottage_blender_light_1.dae" />
+        <mesh filename="package://cottage/meshes/cottage_blender_light_1.dae" />
       </geometry>
     </collision>

File: gazebo/src/cottage/urdf/cottage_blender_light_2.urdf.xacro (robot description, xacro)
@@ -9,5 +9,5 @@
       <origin xyz="0 0 0" rpy="0 0 0" />
       <geometry>
-        <mesh filename="package://cottage_gazebo/meshes/cottage_blender_light_2.dae" />
+        <mesh filename="package://cottage/meshes/cottage_blender_light_2.dae" />
       </geometry>
     </visual>
@@ -15,5 +15,5 @@
       <origin xyz="0 0 0" rpy="0 0 0" />
       <geometry>
-        <mesh filename="package://cottage_gazebo/meshes/cottage_blender_light_2.dae" />
+        <mesh filename="package://cottage/meshes/cottage_blender_light_2.dae" />
       </geometry>
     </collision>

File: gazebo/src/cottage/urdf/cottage_blender_light_3.urdf.xacro (robot description, xacro)
@@ -9,5 +9,5 @@
       <origin xyz="0 0 0" rpy="0 0 0" />
       <geometry>
-        <mesh filename="package://cottage_gazebo/meshes/cottage_blender_light_3.dae" />
+        <mesh filename="package://cottage/meshes/cottage_blender_light_3.dae" />
       </geometry>
     </visual>
@@ -15,5 +15,5 @@
       <origin xyz="0 0 0" rpy="0 0 0" />
       <geometry>
-        <mesh filename="package://cottage_gazebo/meshes/cottage_blender_light_3.dae" />
+        <mesh filename="package://cottage/meshes/cottage_blender_light_3.dae" />
       </geometry>
     </collision>
