Commit message: Loading cottage texture in Docker

File: gazebo/src/cottage/urdf/cottage_blender_ground.urdf.xacro (robot description, xacro)
@@ -20,5 +20,5 @@
   </link>
   <gazebo reference="cottage_blender_ground_link">
-    <material>cottage_texture</material>
+    <material>grass</material>
   </gazebo>
   <gazebo> <static>true</static></gazebo>
